Commit message: LiDAR Tracking - cropMap

File: urdf/lexus.urdf (robot description, URDF)
Before this commit: robot car, 1 links, 0 joints
Links:
- removed link base_link
- added link ego_car; visual mesh filename=package://ndt_localizer/urdf/lexus.dae scale=1.0 1.0 1.0

Commit message: init

File: urdf/lexus.urdf (robot description, URDF)
Before this commit: robot car, 1 links, 0 joints
Links:
- removed link ego_car
- added link base_link; visual mesh filename=package://ndt_localizer/urdf/lexus.dae scale=1.0 1.0 1.0
